File: Null2PowerMod/Null2PowerMod.kicad_pcb (KiCad board)
At the start: 2 copper layers, 18 x 28 mm, 35 parts, among them J1 USB_C_Receptacle_USB2.0, J2 Conn_01x08, J3 Conn_01x01, J4 Conn_01x01, J5 Conn_01x02_Female, U1 TPS61030PWP, U2 MMUN2133LT1G, U3 MCP73871

Commit message: Major revision
Parts:
- removed C3: 2.2 μF, Capacitor_SMD:C_0201_0603Metric
- removed C5: 10μF, Capacitor_SMD:C_0201_0603Metric
- removed D1: Orange, LED_SMD:LED_0201_0603Metric
- removed D2: RED, LED_SMD:LED_0201_0603Metric
- removed D3: BLUE, LED_SMD:LED_0201_0603Metric
- removed D4: Green, LED_SMD:LED_0201_0603Metric
- removed R10: 100k, Resistor_SMD:R_0201_0603Metric
- removed R11, R12: 200k, Resistor_SMD:R_0201_0603Metric
- removed R9: 1k, Resistor_SMD:R_0201_0603Metric
- removed REF** (x2): PinHeader_1x01_P2.54mm_Vertical, Connector_PinHeader_2.54mm:PinHeader_1x01_P2.54mm_Vertical
- removed RT1: NCP15XW153J03RC, NCP15XW153J03RC:THRMC1005X55N
- removed U3: MCP73871, Package_DFN_QFN:QFN-20-1EP_4x4mm_P0.5mm_EP2.5x2.5mm
- added B1: Conn_01x02_Female, Connector_JST:JST_EH_S2B-EH_1x02_P2.50mm_Horizontal, F.Cu at (68.0, 61.5)
- added C7: 10μF, Capacitor_SMD:C_0201_0603Metric, F.Cu at (93.2, 70.4)
- added C8: 10μF, Capacitor_SMD:C_0201_0603Metric, F.Cu at (71.6, 80.4)
- added CHRG/LBO1: ORANGE, LED_SMD:LED_0201_0603Metric, F.Cu at (61.4, 76.9)
- added CN4: USB_C_Receptacle_USB2.0, Connector_USB:USB_C_Receptacle_GCT_USB4085, F.Cu at (66.1, 81.9)
- added Done1: GREEN, LED_SMD:LED_0201_0603Metric, F.Cu at (61.4, 78.2)
- added LED1: RED, LED_SMD:LED_0201_0603Metric, F.Cu at (61.4, 75.5)
- added LED2: BLUE, Capacitor_SMD:C_0201_0603Metric, F.Cu at (61.3, 74.1)
- added R14: 1k, Resistor_SMD:R_0201_0603Metric, F.Cu at (71.4, 69.5)
- added R16: 1k, Resistor_SMD:R_0201_0603Metric, F.Cu at (85.0, 75.5)
- added R17: 100k, Resistor_SMD:R_0201_0603Metric, F.Cu at (99.1, 69.5)
- added R20: 1k, Resistor_SMD:R_0201_0603Metric, F.Cu at (90.8, 70.4)
- added T1: MMUN2133LT1G, ul_MMUN2133LT1G:MMUN2133LT1G, F.Cu at (67.7, 70.8)
- added THERM1: NCP15XW153J03RC, NCP15XW153J03RC:THRMC1005X55N, F.Cu at (74.3, 72.2)
- C1: value 2.2μF -> 10μF
- C2: value 10μF -> 2.2μF
- C4: value 220μF -> 0.1μF; footprint Capacitor_Tantalum_SMD:CP_EIA-2012-15_AVX-P -> Capacitor_SMD:C_0201_0603Metric
- C6: value 10μF -> 100μF
- J1: value USB_C_Receptacle_USB2.0 -> Conn_01x01; footprint Connector_USB:USB_C_Receptacle_GCT_USB4085 -> Connector_PinHeader_2.54mm:PinHeader_1x01_P2.54mm_Vertical
- J5: value Conn_01x02_Female -> Conn_01x01; footprint Connector_JST:JST_EH_S2B-EH_1x02_P2.50mm_Horizontal -> Connector_PinHeader_2.54mm:PinHeader_1x01_P2.54mm_Vertical
- L1: value VLC5045T-330M -> 6.8uH
- R1: value 390kΩ -> 1.87M
- R13: value 1k -> 200k
- R2: value 390kΩ -> 340k
- R3: value 1.05MΩ -> 1.87M
- R4: value 180kΩ -> 200k
- R5: value 1MΩ -> 1k; footprint Resistor_SMD:R_0201_0603Metric -> Capacitor_SMD:C_0201_0603Metric
- R6: value 1k -> 270k
- R7: value 1K -> 100k
- R8: value 270k -> 1k
- U2: value MMUN2133LT1G -> MCP73871; footprint ul_MMUN2133LT1G:MMUN2133LT1G -> Package_DFN_QFN:QFN-20-1EP_4x4mm_P0.5mm_EP2.5x2.5mm
- moved J5 26.1 mm to (76.2, 86.2)
- moved J4 24.4 mm to (61.8, 86.2)
- moved J1 20.5 mm to (61.8, 61.8)
- moved R13 14.4 mm to (74.3, 78.9), turned to 180 degrees
- moved C2 13.5 mm to (74.6, 75.3), turned to 180 degrees
- moved C6 12.7 mm to (81.1, 61.3)
- moved C4 10.1 mm to (85.6, 62.9)
- moved R8 9.33 mm to (81.6, 66.1)
- moved R5 9.28 mm to (79.8, 72.8), turned to 90 degrees
- moved U2 8.03 mm to (72.2, 66.5)
- moved C1 7.55 mm to (64.7, 77.2), turned to 90 degrees
- moved R2 4.14 mm to (64.7, 78.7)
- moved U1 3.69 mm to (69.5, 76.6)
- moved R3 3.42 mm to (74.5, 76.1), turned to 180 degrees
- moved R4 3.23 mm to (74.4, 76.9)
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Connections:
- C1 pad 1: VBUS -> Net-(C1-Pad1)
- C2 pad 1: /Enable -> +5V
- C4 pad 1: +5V -> Net-(C1-Pad1)
- C6 pad 1: VLIPO -> +5V
- J3 pad 1: +5V -> GND
- J4 pad 1: GND -> VBUS
- J5 pad 1: VLIPO -> GND
- L1 pad 1: /Enable -> SW
- L1 pad 2: Net-(L1-Pad2) -> Net-(C1-Pad1)
- R1 pad 1: /Enable -> Net-(C1-Pad1)
- R13 pad 2: Net-(D4-Pad1) -> /Enable
- R5 pad 2: /LB0 -> Net-(LED2-Pad2)
- R6 pad 1: +5V -> VBUS
- R6 pad 2: Net-(D1-Pad2) -> Net-(R6-Pad2)
- R7 pad 1: Net-(R7-Pad1) -> GND
- R7 pad 2: Net-(D2-Pad2) -> Net-(R6-Pad2)
- R8 pad 1: GND -> Net-(R8-Pad1)
- U1 pad 1: Net-(L1-Pad2) -> SW
- U1 pad 10: /LB0 -> Net-(T1-Pad1)
- U1 pad 2: Net-(L1-Pad2) -> SW
- U1 pad 6: /Enable -> Net-(C1-Pad1)
- U2 pad 1: /LB0 -> Net-(U2-Pad1)
- U2 pad 2: Net-(R7-Pad1) -> Net-(R6-Pad2)
- U2 pad 3: Net-(U2-Pad3) -> VBUS
Routing:
- net +5V: track 46.3 -> 0.00 mm, vias 2 -> 0
- net GND: track 43.0 -> 17.9 mm
- net Net-(R13-Pad1): track 24.9 -> 0.00 mm, vias 2 -> 0
- net VBUS: track 60.4 -> 36.7 mm, vias 3 -> 2
- net Net-(R12-Pad1): track 22.8 -> 0.00 mm, vias 2 -> 0
- net /Enable: track 33.3 -> 11.9 mm
- net Net-(R6-Pad2): track 0.00 -> 20.2 mm, vias 0 -> 2
- net VLIPO: track 19.0 -> 0.00 mm
- net Net-(Done1-Pad1): track 0.00 -> 15.7 mm
- net /LB0: track 15.2 -> 0.00 mm, vias 1 -> 0
- net Net-(R7-Pad1): track 14.1 -> 0.00 mm
- net Net-(R11-Pad2): track 12.6 -> 0.00 mm, vias 2 -> 0
- net Net-(L1-Pad2): track 9.59 -> 0.00 mm
- net Net-(R3-Pad2): track 3.62 -> 0.00 mm
- net Net-(C1-Pad1): track 0.00 -> 2.74 mm
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